Commit message: fixing head

File: kit_head_description/model/kit_head.transmission.xacro (robot description, xacro)
@@ -3,7 +3,8 @@
 	<xacro:macro name="kit_head_transmission" params="name">
 		<transmission name="${name}_neck_pitch_joint_trans">
+			<robotNamespace>${name}</robotNamespace>
 			<type>transmission_interface/SimpleTransmission</type>
 			<joint name="${name}_neck_pitch_joint">
-				<hardwareInterface>EffortJointInterface</hardwareInterface>
+				<hardwareInterface>hardware_interface/EffortJointInterface</hardwareInterface>
 			</joint>
 			<actuator name="${name}_neck_pitch_joint_motor">
@@ -12,7 +13,8 @@
 		</transmission>
 		<transmission name="${name}_neck_roll_joint_trans">
+			<robotNamespace>${name}</robotNamespace>
 			<type>transmission_interface/SimpleTransmission</type>
 			<joint name="${name}_neck_roll_joint">
-				<hardwareInterface>EffortJointInterface</hardwareInterface>
+				<hardwareInterface>hardware_interface/EffortJointInterface</hardwareInterface>
 			</joint>
 			<actuator name="${name}_neck_roll_joint_motor">
@@ -21,7 +23,8 @@
 		</transmission>
 		<transmission name="${name}_neck_yaw_joint_trans">
+			<robotNamespace>${name}</robotNamespace>
 			<type>transmission_interface/SimpleTransmission</type>
 			<joint name="${name}_neck_yaw_joint">
-				<hardwareInterface>EffortJointInterface</hardwareInterface>
+				<hardwareInterface>hardware_interface/EffortJointInterface</hardwareInterface>
 			</joint>
 			<actuator name="${name}_neck_yaw_joint_motor">
@@ -30,7 +33,8 @@
 		</transmission>
 		<transmission name="${name}_head_tilt_joint_trans">
+			<robotNamespace>${name}</robotNamespace>
 			<type>transmission_interface/SimpleTransmission</type>
 			<joint name="${name}_head_tilt_joint">
-				<hardwareInterface>EffortJointInterface</hardwareInterface>
+				<hardwareInterface>hardware_interface/EffortJointInterface</hardwareInterface>
 			</joint>
 			<actuator name="${name}_head_tilt_joint_motor">
@@ -39,7 +43,8 @@
 		</transmission>
 		<transmission name="${name}_eyes_tilt_joint_trans">
+			<robotNamespace>${name}</robotNamespace>
 			<type>transmission_interface/SimpleTransmission</type>
 			<joint name="${name}_eyes_tilt_joint">
-				<hardwareInterface>EffortJointInterface</hardwareInterface>
+				<hardwareInterface>hardware_interface/EffortJointInterface</hardwareInterface>
 			</joint>
 			<actuator name="${name}_eyes_tilt_joint_motor">
@@ -48,7 +53,8 @@
 		</transmission>
 		<transmission name="${name}_left_eye_joint_trans">
+			<robotNamespace>${name}</robotNamespace>
 			<type>transmission_interface/SimpleTransmission</type>
 			<joint name="${name}_left_eye_joint">
-				<hardwareInterface>EffortJointInterface</hardwareInterface>
+				<hardwareInterface>hardware_interface/EffortJointInterface</hardwareInterface>
 			</joint>
 			<actuator name="${name}_left_eye_joint_motor">
@@ -57,7 +63,8 @@
 		</transmission>
 		<transmission name="${name}_right_eye_joint_trans">
+			<robotNamespace>${name}</robotNamespace>
 			<type>transmission_interface/SimpleTransmission</type>
 			<joint name="${name}_right_eye_joint">
-				<hardwareInterface>EffortJointInterface</hardwareInterface>
+				<hardwareInterface>hardware_interface/EffortJointInterface</hardwareInterface>
 			</joint>
 			<actuator name="${name}_right_eye_joint_motor">

File: kit_head_description/robot/kit_head.urdf.xacro (robot description, xacro)
@@ -4,5 +4,5 @@
   <link name="world" />
   <xacro:kit_head name="head" parent="world">
-    <origin xyz="0.0 0.0 0.0"/>
+    <origin xyz="0.0 0.0 0.5"/>
   </xacro:kit_head>
 </robot>
