Commit message: adjusting depth sensor urdf

File: kit_head_description/model/kit_head.gazebo.xacro (robot description, xacro)
@@ -140,44 +140,4 @@
 			</sensor>
 		</gazebo>
-		<gazebo reference="${name}_asus_link">
-			<!-- selfCollide>true</selfCollide -->
-			<gravity>true</gravity>
-			<mu1>500.0</mu1>
-			<mu2>500.0</mu2>
-			<kp>10000000.0</kp>
-			<kd>1.0</kd>
-			<sensor type="depth" name="${name}_xtion">
-				<update_rate>10</update_rate>
-				<camera>
-					<horizontal_fov>1.09606677025</horizontal_fov>
-					<image>
-						<format>R8G8B8</format>
-						<width>640</width>
-						<height>480</height>
-					</image>
-					<clip>
-						<near>0.5</near>
-						<far>9</far>
-					</clip>
-				</camera>
-				<plugin filename="libgazebo_ros_openni_kinect.so" name="xtion_camera_controller">
-					<alwaysOn>true</alwaysOn>
-					<updateRate>10</updateRate>
-					<cameraName>${name}_asus</cameraName>
-					<imageTopicName>${name}_asus/rgb/image_raw</imageTopicName>
-					<cameraInfoTopicName>${name}_asus/rgb/camera_info</cameraInfoTopicName>
-					<depthImageTopicName>${name}_asus/depth/image_raw</depthImageTopicName>
-					<depthImageCameraInfoTopicName>${name}_asus/depth/camera_info</depthImageCameraInfoTopicName>
-					<pointCloudTopicName>${name}_asus/depth/points</pointCloudTopicName>
-					<frameName>${name}_asus/camera_rgb_optical_frame</frameName>
-					<pointCloudCutoff>0.5</pointCloudCutoff>
-					<distortion_k1>0.0</distortion_k1>
-					<distortion_k2>0.0</distortion_k2>
-					<distortion_k3>0.0</distortion_k3>
-					<distortion_t1>0.0</distortion_t1>
-					<distortion_t2>0.0</distortion_t2>
-				</plugin>
-			</sensor>
-		</gazebo>
 		<!-- plugin name="${name}_asus_controller" filename="libgazebo_ros_openni_kinect.so">
 			<baseline>0.2</baseline>

File: kit_head_description/model/kit_head.urdf.xacro (robot description, xacro)
@@ -5,4 +5,5 @@
   <xacro:include filename="$(find kit_head_description)/model/kit_head.transmission.xacro"/>
   <xacro:include filename="$(find kit_head_description)/model/kit_head.gazebo.xacro"/>
+  <xacro:include filename="$(find kit_head_description)/model/depth_sensor.gazebo.xacro"/>
   <xacro:property name="M_PI" value="3.1415926535897931" />
   <xacro:property name="velocity_scale_factor" value="1.0"/>
@@ -293,6 +294,32 @@
       </collision>
     </link>
+      <!-- ASUS Xtion -->
+    <link name="${name}_camera_depth_frame"/>
+    <link name="${name}_camera_rgb_frame"/>
+    <link name="${name}_camera_depth_optical_frame"/>
+    <link name="${name}_camera_rgb_optical_frame"/>
+    <joint name="${name}_camera_depth_frame_joint" type="fixed" >
+      <origin rpy="0 0 0" xyz="0 0.045 0.02" />
+      <parent link="${name}_asus_link"/>
+      <child link="${name}_camera_depth_frame"/>
+    </joint>
+    <joint name="${name}_camera_rgb_frame_joint" type="fixed">
+      <origin rpy="0.0 0.0 0.0" xyz="0 0.02 0.02"/>
+      <parent link="${name}_asus_link"/>
+      <child link="${name}_camera_rgb_frame"/>
+    </joint>
+    <joint name="${name}_camera_depth_optical_frame_joint" type="fixed" >
+      <origin rpy="${-M_PI/2} 0 ${-M_PI/2}" xyz="0 0 0" />
+      <parent link="${name}_camera_depth_frame"/>
+      <child link="${name}_camera_depth_optical_frame"/>
+    </joint>
+    <joint name="${name}_camera_rgb_optical_frame_joint" type="fixed" >
+      <origin rpy="${-M_PI/2} 0 ${-M_PI/2}" xyz="0 0 0" />
+      <parent link="${name}_camera_rgb_frame"/>
+      <child link="${name}_camera_rgb_optical_frame"/>
+    </joint>
     <xacro:kit_head_transmission name="${name}"/>
     <xacro:kit_head_gazebo name="${name}"/>
+    <xacro:head_depth_sensor name="${name}" parent="${name}_asus_link"/>
   </xacro:macro>
 </robot>

Commit message: updates to ros kinetic

File: kit_head_description/model/kit_head.gazebo.xacro (robot description, xacro)
@@ -1,4 +1,4 @@
 <?xml version="1.0"?>
-<robot xmlns:xacro="http://ros.org/wiki/xacro">
+<robot xmlns:xacro="http://www.ros.org/wiki/xacro">
 	<xacro:macro name="kit_head_gazebo" params="name">
 		<gazebo reference="${name}_base_link">
@@ -140,44 +140,4 @@
 			</sensor>
 		</gazebo>
-		<gazebo reference="${name}_asus_link">
-			<!-- selfCollide>true</selfCollide -->
-			<gravity>true</gravity>
-			<mu1>500.0</mu1>
-			<mu2>500.0</mu2>
-			<kp>10000000.0</kp>
-			<kd>1.0</kd>
-			<sensor type="depth" name="${name}_xtion">
-				<update_rate>10</update_rate>
-				<camera>
-					<horizontal_fov>1.09606677025</horizontal_fov>
-					<image>
-						<format>R8G8B8</format>
-						<width>640</width>
-						<height>480</height>
-					</image>
-					<clip>
-						<near>0.5</near>
-						<far>9</far>
-					</clip>
-				</camera>
-				<plugin filename="libgazebo_ros_openni_kinect.so" name="xtion_camera_controller">
-					<alwaysOn>true</alwaysOn>
-					<updateRate>10</updateRate>
-					<cameraName>${name}_asus</cameraName>
-					<imageTopicName>${name}_asus/rgb/image_raw</imageTopicName>
-					<cameraInfoTopicName>${name}_asus/rgb/camera_info</cameraInfoTopicName>
-					<depthImageTopicName>${name}_asus/depth/image_raw</depthImageTopicName>
-					<depthImageCameraInfoTopicName>${name}_asus/depth/camera_info</depthImageCameraInfoTopicName>
-					<pointCloudTopicName>${name}_asus/depth_registered/points</pointCloudTopicName>
-					<frameName>${name}_asus/camera_rgb_optical_frame</frameName>
-					<pointCloudCutoff>0.5</pointCloudCutoff>
-					<distortion_k1>0.0</distortion_k1>
-					<distortion_k2>0.0</distortion_k2>
-					<distortion_k3>0.0</distortion_k3>
-					<distortion_t1>0.0</distortion_t1>
-					<distortion_t2>0.0</distortion_t2>
-				</plugin>
-			</sensor>
-		</gazebo>
 		<!-- plugin name="${name}_asus_controller" filename="libgazebo_ros_openni_kinect.so">
 			<baseline>0.2</baseline>
@@ -204,5 +164,5 @@
 		</plugin -->
 		<gazebo>
-			<plugin name="${name}_kit_head_hw_sim_plugin" filename="libkit_head_hw_sim_plugin.so">
+			<plugin name="gazebo_ros_control" filename="libgazebo_ros_control.so">
 				<robotNamespace>${name}</robotNamespace>
 			</plugin>

File: kit_head_description/model/kit_head.inertia.xacro (robot description, xacro)
@@ -1,4 +1,4 @@
 <?xml version="1.0"?>
-<robot xmlns:xacro="http://ros.org/wiki/xacro">
+<robot xmlns:xacro="http://www.ros.org/wiki/xacro">
     <!-- NOTE: inertia values are approximated using meshlab and only using the significant elements -->
     <!-- from http://answers.ros.org/question/11350/is-there-any-way-to-calculate-inertial-property-of-a-robot-to-simulate-it-in-gazebo/s

File: kit_head_description/model/kit_head.transmission.xacro (robot description, xacro)
@@ -3,8 +3,7 @@
 	<xacro:macro name="kit_head_transmission" params="name">
 		<transmission name="${name}_neck_pitch_joint_trans">
-			<robotNamespace>${name}</robotNamespace>
 			<type>transmission_interface/SimpleTransmission</type>
 			<joint name="${name}_neck_pitch_joint">
-				<hardwareInterface>PositionJointInterface</hardwareInterface>
+				<hardwareInterface>EffortJointInterface</hardwareInterface>
 			</joint>
 			<actuator name="${name}_neck_pitch_joint_motor">
@@ -13,8 +12,7 @@
 		</transmission>
 		<transmission name="${name}_neck_roll_joint_trans">
-			<robotNamespace>${name}</robotNamespace>
 			<type>transmission_interface/SimpleTransmission</type>
 			<joint name="${name}_neck_roll_joint">
-				<hardwareInterface>PositionJointInterface</hardwareInterface>
+				<hardwareInterface>EffortJointInterface</hardwareInterface>
 			</joint>
 			<actuator name="${name}_neck_roll_joint_motor">
@@ -23,8 +21,7 @@
 		</transmission>
 		<transmission name="${name}_neck_yaw_joint_trans">
-			<robotNamespace>${name}</robotNamespace>
 			<type>transmission_interface/SimpleTransmission</type>
 			<joint name="${name}_neck_yaw_joint">
-				<hardwareInterface>PositionJointInterface</hardwareInterface>
+				<hardwareInterface>EffortJointInterface</hardwareInterface>
 			</joint>
 			<actuator name="${name}_neck_yaw_joint_motor">
@@ -33,8 +30,7 @@
 		</transmission>
 		<transmission name="${name}_head_tilt_joint_trans">
-			<robotNamespace>${name}</robotNamespace>
 			<type>transmission_interface/SimpleTransmission</type>
 			<joint name="${name}_head_tilt_joint">
-				<hardwareInterface>PositionJointInterface</hardwareInterface>
+				<hardwareInterface>EffortJointInterface</hardwareInterface>
 			</joint>
 			<actuator name="${name}_head_tilt_joint_motor">
@@ -43,8 +39,7 @@
 		</transmission>
 		<transmission name="${name}_eyes_tilt_joint_trans">
-			<robotNamespace>${name}</robotNamespace>
 			<type>transmission_interface/SimpleTransmission</type>
 			<joint name="${name}_eyes_tilt_joint">
-				<hardwareInterface>PositionJointInterface</hardwareInterface>
+				<hardwareInterface>EffortJointInterface</hardwareInterface>
 			</joint>
 			<actuator name="${name}_eyes_tilt_joint_motor">
@@ -53,8 +48,7 @@
 		</transmission>
 		<transmission name="${name}_left_eye_joint_trans">
-			<robotNamespace>${name}</robotNamespace>
 			<type>transmission_interface/SimpleTransmission</type>
 			<joint name="${name}_left_eye_joint">
-				<hardwareInterface>PositionJointInterface</hardwareInterface>
+				<hardwareInterface>EffortJointInterface</hardwareInterface>
 			</joint>
 			<actuator name="${name}_left_eye_joint_motor">
@@ -63,8 +57,7 @@
 		</transmission>
 		<transmission name="${name}_right_eye_joint_trans">
-			<robotNamespace>${name}</robotNamespace>
 			<type>transmission_interface/SimpleTransmission</type>
 			<joint name="${name}_right_eye_joint">
-				<hardwareInterface>PositionJointInterface</hardwareInterface>
+				<hardwareInterface>EffortJointInterface</hardwareInterface>
 			</joint>
 			<actuator name="${name}_right_eye_joint_motor">

File: kit_head_description/model/kit_head.urdf.xacro (robot description, xacro)
@@ -5,4 +5,5 @@
   <xacro:include filename="$(find kit_head_description)/model/kit_head.transmission.xacro"/>
   <xacro:include filename="$(find kit_head_description)/model/kit_head.gazebo.xacro"/>
+  <xacro:include filename="$(find kit_head_description)/model/depth_sensor.gazebo.xacro"/>
   <xacro:property name="M_PI" value="3.1415926535897931" />
   <xacro:property name="velocity_scale_factor" value="1.0"/>
@@ -10,5 +11,5 @@
     <!-- The base of the hand, fixed to its parent. -->
     <joint name="${parent}_${name}_base_joint" type="fixed">
-      <insert_block name="origin"/>
+      <xacro:insert_block name="origin"/>
       <parent link="${parent}"/>
       <child link="${name}_base_link"/>
@@ -16,5 +17,5 @@
     <link name="${name}_base_link">
       <inertial>
-        <insert_block name="negligible_inertia"/>
+        <xacro:insert_block name="negligible_inertia"/>
       </inertial>
       <!-- <visual>
@@ -48,5 +49,5 @@
     <link name="${name}_head_1_link">
       <inertial>
-        <insert_block name="negligible_inertia"/>
+        <xacro:insert_block name="negligible_inertia"/>
       </inertial>
       <visual>
@@ -79,5 +80,5 @@
     <link name="${name}_head_2_link">
       <inertial>
-        <insert_block name="negligible_inertia"/>
+        <xacro:insert_block name="negligible_inertia"/>
       </inertial>
       <visual>
@@ -110,5 +111,5 @@
     <link name="${name}_head_3_link">
       <inertial>
-        <insert_block name="negligible_inertia"/>
+        <xacro:insert_block name="negligible_inertia"/>
       </inertial>
       <visual>
@@ -141,5 +142,5 @@
     <link name="${name}_head_4_link">
       <inertial>
-        <insert_block name="negligible_inertia"/>
+        <xacro:insert_block name="negligible_inertia"/>
       </inertial>
       <visual>
@@ -172,5 +173,5 @@
     <link name="${name}_head_5_link">
       <inertial>
-        <insert_block name="negligible_inertia"/>
+        <xacro:insert_block name="negligible_inertia"/>
       </inertial>
       <visual>
@@ -203,5 +204,5 @@
     <link name="${name}_left_eye_link">
       <inertial>
-        <insert_block name="negligible_inertia"/>
+        <xacro:insert_block name="negligible_inertia"/>
       </inertial>
       <visual>
@@ -234,5 +235,5 @@
     <link name="${name}_right_eye_link">
       <inertial>
-        <insert_block name="negligible_inertia"/>
+        <xacro:insert_block name="negligible_inertia"/>
       </inertial>
       <visual>
@@ -277,5 +278,5 @@
     <link name="${name}_asus_link">
       <inertial>
-        <insert_block name="negligible_inertia"/>
+        <xacro:insert_block name="negligible_inertia"/>
       </inertial>
       <visual>
@@ -293,6 +294,32 @@
       </collision>
     </link>
+      <!-- ASUS Xtion -->
+    <link name="${name}_camera_depth_frame"/>
+    <link name="${name}_camera_rgb_frame"/>
+    <link name="${name}_camera_depth_optical_frame"/>
+    <link name="${name}_camera_rgb_optical_frame"/>
+    <joint name="${name}_camera_depth_frame_joint" type="fixed" >
+      <origin rpy="0 0 0" xyz="0 0.045 0.02" />
+      <parent link="${name}_asus_link"/>
+      <child link="${name}_camera_depth_frame"/>
+    </joint>
+    <joint name="${name}_camera_rgb_frame_joint" type="fixed">
+      <origin rpy="0.0 0.0 0.0" xyz="0 0.02 0.02"/>
+      <parent link="${name}_asus_link"/>
+      <child link="${name}_camera_rgb_frame"/>
+    </joint>
+    <joint name="${name}_camera_depth_optical_frame_joint" type="fixed" >
+      <origin rpy="${-M_PI/2} 0 ${-M_PI/2}" xyz="0 0 0" />
+      <parent link="${name}_camera_depth_frame"/>
+      <child link="${name}_camera_depth_optical_frame"/>
+    </joint>
+    <joint name="${name}_camera_rgb_optical_frame_joint" type="fixed" >
+      <origin rpy="${-M_PI/2} 0 ${-M_PI/2}" xyz="0 0 0" />
+      <parent link="${name}_camera_rgb_frame"/>
+      <child link="${name}_camera_rgb_optical_frame"/>
+    </joint>
     <xacro:kit_head_transmission name="${name}"/>
     <xacro:kit_head_gazebo name="${name}"/>
+    <xacro:head_depth_sensor name="${name}" parent="${name}_asus_link"/>
   </xacro:macro>
 </robot>

Commit message: simulated kit-head, albeit hack at the moment

File: kit_head_description/model/kit_head.gazebo.xacro (robot description, xacro)
@@ -164,6 +164,8 @@
 		</plugin -->
 		<gazebo>
-			<plugin name="gazebo_ros_control" filename="libgazebo_ros_control.so">
+			<plugin name="kit_head_gazebo_ros_control" filename="libkit_head_gazebo_ros_control.so">
 				<robotNamespace>${name}</robotNamespace>
+				<robotSimType>kit_head_hw/DefaultKITHeadHWSim</robotSimType>
+				<legacyModeNS>false</legacyModeNS>
 			</plugin>
 		</gazebo>

File: kit_head_description/model/kit_head.transmission.xacro (robot description, xacro)
@@ -2,9 +2,12 @@
 <robot name="robot" xmlns:xacro="http://www.ros.org/wiki/xacro">
 	<xacro:macro name="kit_head_transmission" params="name">
+		<xacro:property name="Interface10" value="hardware_interface/PositionJointInterface"/>
+		<xacro:property name="Interface30" value="hardware_interface/EffortJointInterface"/>
 		<transmission name="${name}_neck_pitch_joint_trans">
 			<robotNamespace>${name}</robotNamespace>
 			<type>transmission_interface/SimpleTransmission</type>
 			<joint name="${name}_neck_pitch_joint">
-				<hardwareInterface>hardware_interface/EffortJointInterface</hardwareInterface>
+				<hardwareInterface>${Interface10}</hardwareInterface>
+				<!-- <hardwareInterface>${Interface30}</hardwareInterface> -->
 			</joint>
 			<actuator name="${name}_neck_pitch_joint_motor">
@@ -16,5 +19,6 @@
 			<type>transmission_interface/SimpleTransmission</type>
 			<joint name="${name}_neck_roll_joint">
-				<hardwareInterface>hardware_interface/EffortJointInterface</hardwareInterface>
+				<hardwareInterface>${Interface10}</hardwareInterface>
+				<!-- <hardwareInterface>${Interface30}</hardwareInterface> -->
 			</joint>
 			<actuator name="${name}_neck_roll_joint_motor">
@@ -26,5 +30,6 @@
 			<type>transmission_interface/SimpleTransmission</type>
 			<joint name="${name}_neck_yaw_joint">
-				<hardwareInterface>hardware_interface/EffortJointInterface</hardwareInterface>
+				<hardwareInterface>${Interface10}</hardwareInterface>
+				<!-- <hardwareInterface>${Interface30}</hardwareInterface> -->
 			</joint>
 			<actuator name="${name}_neck_yaw_joint_motor">
@@ -36,5 +41,6 @@
 			<type>transmission_interface/SimpleTransmission</type>
 			<joint name="${name}_head_tilt_joint">
-				<hardwareInterface>hardware_interface/EffortJointInterface</hardwareInterface>
+				<hardwareInterface>${Interface10}</hardwareInterface>
+				<!-- <hardwareInterface>${Interface30}</hardwareInterface> -->
 			</joint>
 			<actuator name="${name}_head_tilt_joint_motor">
@@ -46,5 +52,6 @@
 			<type>transmission_interface/SimpleTransmission</type>
 			<joint name="${name}_eyes_tilt_joint">
-				<hardwareInterface>hardware_interface/EffortJointInterface</hardwareInterface>
+				<hardwareInterface>${Interface10}</hardwareInterface>
+				<!-- <hardwareInterface>${Interface30}</hardwareInterface> -->
 			</joint>
 			<actuator name="${name}_eyes_tilt_joint_motor">
@@ -56,5 +63,6 @@
 			<type>transmission_interface/SimpleTransmission</type>
 			<joint name="${name}_left_eye_joint">
-				<hardwareInterface>hardware_interface/EffortJointInterface</hardwareInterface>
+				<hardwareInterface>${Interface10}</hardwareInterface>
+				<!-- <hardwareInterface>${Interface30}</hardwareInterface> -->
 			</joint>
 			<actuator name="${name}_left_eye_joint_motor">
@@ -66,5 +74,6 @@
 			<type>transmission_interface/SimpleTransmission</type>
 			<joint name="${name}_right_eye_joint">
-				<hardwareInterface>hardware_interface/EffortJointInterface</hardwareInterface>
+				<hardwareInterface>${Interface10}</hardwareInterface>
+				<!-- <hardwareInterface>${Interface30}</hardwareInterface> -->
 			</joint>
 			<actuator name="${name}_right_eye_joint_motor">
